File: Eagle files/v1.1/jefboard1.1.brd (EAGLE design)
At the start: 60.6 x 40.6 mm, 20 parts, among them IC1 ATtiny2313, IC2 LM1117DTX-3.3

Commit message: ...
Connections:
- net N$1: now also IC2.TAB
